File: _hardware/pcb/tergo-kailh/tergo-kailh.kicad_sch (KiCad schematic)
At the start: 131 parts, among them J1 TRRS, J2 Conn_01x04_Socket, J3 Conn_01x04_Socket, Q1 FDN335N, SW1 SW_Push, SW10 SW_Push, SW11 SW_Push, SW12 SW_Push, SW13 SW_Push, SW14 SW_Push, SW15 SW_Push, SW16 SW_Push, SW17 SW_Push, SW18 SW_Push, SW19 SW_Push, SW2 SW_Push, SW20 SW_Push, SW21 SW_Push, SW22 SW_Push, SW23 SW_Push, SW24 SW_Push, SW25 SW_Push, SW26 SW_Push, SW27 SW_Push, SW28 SW_Push, SW29 SW_Push, SW3 SW_Push, SW4 SW_Push, SW5 SW_Push, SW6 SW_Push, SW7 SW_Push, SW8 SW_Push, SW9 SW_Push, U1 Raspberry_Pi_Pico

Commit message: wip
Parts:
- removed D1, D10, D11, D12, D13, D14, D15, D16, D17, D18, D19, D2, D20, D21, D22, D23, D24, D25, D26, D27, D28, D3, D4, D5, D6, D7, D8, D9: D_Small, _tergo_lib:Diode-Hybrid-2sided, symbol Device:D_Small
- removed D29, D30, D31, D32, D33, D34, D35, D36, D37, D38, D39, D40, D41, D42, D43, D44, D45, D46, D47, D48, D49, D50, D51, D52, D53, D54, D55, D56: LED_Small, _tergo_lib:LED_1.8mm, symbol Device:LED_Small
- removed H1, H2, H3, H4, H5, H6, H7, H8, H9: CaseHole, _tergo_lib:MountHole, symbol Mechanical:MountingHole
- removed J1: TRRS, _tergo_lib:MJ-4PP-9-mirrored, symbol _tergo_lib:MJ-4PP-9
- removed J2, J3: Conn_01x04_Socket, Connector_PinHeader_2.54mm:PinHeader_1x04_P2.54mm_Vertical, symbol Connector:Conn_01x04_Socket
- removed JP1: Jumper_3_Open, Jumper:SolderJumper-3_P1.3mm_Open_RoundedPad1.0x1.5mm, symbol Jumper:Jumper_3_Open
- removed JPL1, JPR2: Jumper_2_Open, Jumper:SolderJumper-2_P1.3mm_Open_RoundedPad1.0x1.5mm, symbol Jumper:Jumper_2_Open
- removed Q1: FDN335N, Package_TO_SOT_SMD:SOT-23, symbol Transistor_FET:2N7002
- removed R1, R10, R11, R12, R13, R14, R15, R16, R17, R18, R19, R2, R20, R21, R22, R23, R24, R25, R26, R27, R3, R4, R5, R6, R7, R8, R9: R_Small, _tergo_lib:Resistor-Hybrid-2sided, symbol Device:R_Small
- removed R31: 10k, _tergo_lib:Resistor-Hybrid-2sided, symbol Device:R_Small
- removed SW1, SW10, SW11, SW12, SW13, SW14, SW15, SW16, SW17, SW18, SW19, SW2, SW20, SW21, SW22, SW23, SW24, SW25, SW26, SW27, SW28, SW3, SW4, SW5, SW6, SW7, SW8, SW9: SW_Push, _tergo_lib:SW_Hotswap_Kailh_MX_Plated_mirrored2_1.00u, symbol Switch:SW_Push
- removed SW29: SW_Push, _tergo_lib:ResetSW, symbol Switch:SW_Push
- removed U1: Raspberry_Pi_Pico, _tergo_lib:Raspberry_Pi_Pico_dual, symbol _tergo_lib:Raspberry_Pi_Pico
- added D116, D117, D118, D119, D120, D121, D122, D123, D125, D126, D127, D128, D129, D130, D131, D132, D133, D134, D135, D136, D137, D138, D139, D140, D141, D142, D143, D144, D145, D146, D147, D148, D149, D150, D151, D152, D153, D154, D155, D156, D157, D158, D159, D160, D161, D162, D163, D164, D165, D166, D167, D168, D169, D170, D171, D53: D_Small, symbol Device:D_Small
- added D124: LED_Small, _tergo_lib:LED_1.8mm, symbol Device:LED_Small
- added J10: Conn_01x04_Socket, Connector_PinHeader_2.54mm:PinHeader_1x04_P2.54mm_Vertical, symbol Connector:Conn_01x04_Socket
- added J5: TRRS, _tergo_lib:MJ-4PP-9, symbol _tergo_lib:MJ-4PP-9
- added SW116, SW117, SW118, SW119, SW120, SW121, SW122, SW123, SW124, SW125, SW126, SW127, SW128, SW129, SW130, SW131, SW132, SW133, SW134, SW135, SW136, SW137, SW138, SW139, SW140, SW141, SW142, SW143, SW144, SW145, SW146, SW147, SW148, SW149, SW150, SW151, SW152, SW153, SW154, SW155, SW156, SW157, SW158, SW159, SW160, SW161, SW162, SW163, SW164, SW165, SW166, SW167, SW168, SW169, SW170, SW171, SW172: SW_Push, symbol Switch:SW_Push
- added U4: Raspberry_Pi_Pico, _tergo_lib:Raspberry_Pi_Pico_dual, symbol _tergo_lib:Raspberry_Pi_Pico
- R28: footprint _tergo_lib:Resistor-Hybrid-2sided -> Resistor_SMD:R_0805_2012Metric_Pad1.20x1.40mm_HandSolder
Connections:
- net LEDOut is gone; now on net GND: R28.2
- net 3V3: now also J10.2 (Pin_2), U4.36 (3V3)
- net DISPLAY_SCL: now also J10.3 (Pin_3), U4.22 (GP17/SCL)
- net DISPLAY_SDA: now also J10.4 (Pin_4), U4.21 (GP16/SDA)
- net GND: now also J10.1 (Pin_1), J5.A, SW116.2, U4.13 (GND), U4.18 (GND), U4.23 (GND), U4.28 (GND), U4.29 (GP22), U4.3 (GND), U4.33 (AGND), U4.38 (GND), U4.8 (GND)
- net RX: now also J5.B, U4.2RXL (GP1/RX)
- net TX: now also J5.C, U4.1TXL (GP0/TX)
- net Vin: now also J5.DR, U4.39 (Vin)
- net Vout: now also J5.DL, U4.40 (Vout)
- net col0: now also SW117.2, SW118.2, SW119.2, SW120.2, SW121.2, SW145.2, SW146.2, SW147.2, SW148.2, SW149.2, U4.4 (GP2)
- net col1: now also SW122.2, SW123.2, SW124.2, SW125.2, SW150.2, SW151.2, SW152.2, SW153.2, U4.7 (GP5)
- net col2: now also SW126.2, SW127.2, SW128.2, SW129.2, SW154.2, SW155.2, SW156.2, SW157.2, U4.6 (GP4)
- net col3: now also SW130.2, SW131.2, SW132.2, SW133.2, SW134.2, SW158.2, SW159.2, SW160.2, SW161.2, SW162.2, U4.10 (GP7)
- net col4: now also SW135.2, SW136.2, SW137.2, SW138.2, SW139.2, SW163.2, SW164.2, SW165.2, SW166.2, SW167.2, U4.11 (GP8)
- net col5: now also SW140.2, SW141.2, SW142.2, SW143.2, SW144.2, SW168.2, SW169.2, SW170.2, SW171.2, SW172.2, U4.12 (GP9)
- net rowA: now also D120.1 (K), D125.1 (K), D129.1 (K), D134.1 (K), D139.1 (K), D144.1 (K), D149.1 (K), D153.1 (K), D157.1 (K), D162.1 (K), D167.1 (K), D53.1 (K), U4.5 (GP3)
- net rowB: now also D116.1 (K), D121.1 (K), D126.1 (K), D130.1 (K), D135.1 (K), D140.1 (K), D145.1 (K), D150.1 (K), D154.1 (K), D158.1 (K), D163.1 (K), D168.1 (K), U4.9 (GP6)
- net rowC: now also D117.1 (K), D122.1 (K), D127.1 (K), D131.1 (K), D136.1 (K), D141.1 (K), D146.1 (K), D151.1 (K), D155.1 (K), D159.1 (K), D164.1 (K), D169.1 (K), U4.16 (GP12)
- net rowD: now also D118.1 (K), D123.1 (K), D128.1 (K), D132.1 (K), D137.1 (K), D142.1 (K), D147.1 (K), D152.1 (K), D156.1 (K), D160.1 (K), D165.1 (K), D170.1 (K), U4.17 (GP13)
- net rowE: now also D119.1 (K), D133.1 (K), D138.1 (K), D143.1 (K), D148.1 (K), D161.1 (K), D166.1 (K), D171.1 (K), U4.19 (GP14)
- net at R28.1: now also D124.1 (K)
- new net: D151.2 (A), SW152.1
- new net: D163.2 (A), SW164.1
- new net: D135.2 (A), SW136.1
- new net: D133.2 (A), SW134.1
- new net: D161.2 (A), SW162.1
- new net: D158.2 (A), SW159.1
- new net: D142.2 (A), SW143.1
- new net: D119.2 (A), SW121.1
- new net: D140.2 (A), SW141.1
- new net: D171.2 (A), SW172.1
- new net: D53.2 (A), SW117.1
- new net: D126.2 (A), SW127.1
- new net: D143.2 (A), SW144.1
- new net: D122.2 (A), SW124.1
- new net: D153.2 (A), SW154.1
- new net: D156.2 (A), SW157.1
- new net: D168.2 (A), SW169.1
- new net: D160.2 (A), SW161.1
- new net: D117.2 (A), SW119.1
- new net: D146.2 (A), SW147.1
- new net: D147.2 (A), SW148.1
- new net: D164.2 (A), SW165.1
- new net: D123.2 (A), SW125.1
- new net: D120.2 (A), SW122.1
- new net: D169.2 (A), SW170.1
- new net: D131.2 (A), SW132.1
- new net: D136.2 (A), SW137.1
- new net: D167.2 (A), SW168.1
- new net: D165.2 (A), SW166.1
- new net: D129.2 (A), SW130.1
- new net: D154.2 (A), SW155.1
- new net: D150.2 (A), SW151.1
- new net: D121.2 (A), SW123.1
- new net: D166.2 (A), SW167.1
- new net: D134.2 (A), SW135.1
- new net: D144.2 (A), SW145.1
- new net: D130.2 (A), SW131.1
- new net: D137.2 (A), SW138.1
- new net: D145.2 (A), SW146.1
- new net: D138.2 (A), SW139.1
- new net: D149.2 (A), SW150.1
- new net: D157.2 (A), SW158.1
- new net: D170.2 (A), SW171.1
- new net: D118.2 (A), SW120.1
- new net: D148.2 (A), SW149.1
- new net: D159.2 (A), SW160.1
- new net: D139.2 (A), SW140.1
- new net: D155.2 (A), SW156.1
- new net: D132.2 (A), SW133.1
- new net: D141.2 (A), SW142.1
- new net: D128.2 (A), SW129.1
- new net: D127.2 (A), SW128.1
- new net: D116.2 (A), SW118.1
- new net: D125.2 (A), SW126.1
- new net: D162.2 (A), SW163.1
- new net: D152.2 (A), SW153.1
- new net LED_L: D124.2 (A), U4.20 (GP15)
- new net RST_L: SW116.1, U4.30 (RUN)
