File: hardware/pcb/tergo-choc/tergo-choc.kicad_sch (KiCad schematic)
At the start: 118 parts, among them J10 Conn_01x04_Socket, J5 TRRS, SW116 SW_Push, SW117 SW_Push, SW118 SW_Push, SW119 SW_Push, SW120 SW_Push, SW121 SW_Push, SW122 SW_Push, SW123 SW_Push, SW124 SW_Push, SW125 SW_Push, SW126 SW_Push, SW127 SW_Push, SW128 SW_Push, SW129 SW_Push, SW130 SW_Push, SW131 SW_Push, SW132 SW_Push, SW133 SW_Push, SW134 SW_Push, SW135 SW_Push, SW136 SW_Push, SW137 SW_Push, SW138 SW_Push, SW139 SW_Push, SW140 SW_Push, SW141 SW_Push, SW142 SW_Push, SW143 SW_Push, SW144 SW_Push, SW145 SW_Push, SW146 SW_Push, SW147 SW_Push, SW148 SW_Push, SW149 SW_Push, SW150 SW_Push, SW151 SW_Push, SW152 SW_Push, SW153 SW_Push, SW154 SW_Push, SW155 SW_Push, SW156 SW_Push, SW157 SW_Push, SW158 SW_Push, SW159 SW_Push, SW160 SW_Push, SW161 SW_Push, SW162 SW_Push, SW163 SW_Push, SW164 SW_Push, SW165 SW_Push, SW166 SW_Push, SW167 SW_Push, SW168 SW_Push, SW169 SW_Push, SW170 SW_Push, SW171 SW_Push, SW172 SW_Push, U4 Raspberry_Pi_Pico

Commit message: wip
Parts:
- added D59, D60: LED_Small, _tergo_lib:LED_1.8mm, symbol Device:LED_Small
- added J3: TRRS, _tergo_lib:MJ-4PP-9, symbol _tergo_lib:MJ-4PP-9
- added R3, R4: R_Small, Resistor_SMD:R_0805_2012Metric_Pad1.20x1.40mm_HandSolder, symbol Device:R_Small
- added SW30: SW_Push, symbol Switch:SW_Push
- added U2: Raspberry_Pi_Pico, _tergo_lib:Raspberry_Pi_Pico, symbol _tergo_lib:Raspberry_Pi_Pico
- U1: renamed from U4; footprint _tergo_lib:Raspberry_Pi_Pico_dual -> _tergo_lib:Raspberry_Pi_Pico
- renumbered D53 to D1, D124 to D10, D125 to D11, D126 to D12, D127 to D13, D128 to D14, D129 to D15, D130 to D16, D131 to D17, D132 to D18, D133 to D19, D116 to D2, D134 to D20, D135 to D21, D136 to D22, D137 to D23, D138 to D24, D139 to D25, D140 to D26, D141 to D27, D142 to D28, D143 to D29, D117 to D3, D144 to D30, D145 to D31, D146 to D32, D147 to D33, D148 to D34, D149 to D35, D150 to D36, D151 to D37, D152 to D38, D153 to D39, D118 to D4, D154 to D40, D155 to D41, D156 to D42, D157 to D44, D158 to D45, D159 to D46, D160 to D47, D161 to D48, D162 to D49, D119 to D5, D163 to D50, D164 to D51, D165 to D52, D166 to D53, D167 to D54, D168 to D55, D169 to D56, D170 to D57, D171 to D58, D120 to D6, D121 to D7, D122 to D8, D123 to D9, J5 to J1, J10 to J2, R28 to R1, SW116 to SW1, SW125 to SW10, SW126 to SW11, SW127 to SW12, SW128 to SW13, SW129 to SW14, SW130 to SW15, SW131 to SW16, SW132 to SW17, SW133 to SW18, SW134 to SW19, SW117 to SW2, SW135 to SW20, SW136 to SW21, SW137 to SW22, SW138 to SW23, SW139 to SW24, SW140 to SW25, SW141 to SW26, SW142 to SW27, SW143 to SW28, SW144 to SW29, SW118 to SW3, SW145 to SW31, SW146 to SW32, SW147 to SW33, SW148 to SW34, SW149 to SW35, SW150 to SW36, SW151 to SW37, SW152 to SW38, SW153 to SW39, SW119 to SW4, SW154 to SW40, SW155 to SW41, SW156 to SW42, SW157 to SW43, SW158 to SW44, SW159 to SW45, SW160 to SW46, SW161 to SW47, SW162 to SW48, SW163 to SW49, SW120 to SW5, SW164 to SW50, SW165 to SW51, SW166 to SW52, SW167 to SW53, SW168 to SW54, SW169 to SW55, SW170 to SW56, SW171 to SW57, SW172 to SW58, SW121 to SW6, SW122 to SW7, SW123 to SW8, SW124 to SW9
Connections:
- net 3V3: now also U2.36 (3V3)
- net DISPLAY_SCL: now also U2.22 (GP17/SCL)
- net DISPLAY_SDA: now also U2.21 (GP16/SDA)
- net GND: now also J3.A, R3.2, R4.2, SW30.2, U2.13 (GND), U2.18 (GND), U2.23 (GND), U2.28 (GND), U2.29 (GP22), U2.3 (GND), U2.33 (AGND), U2.38 (GND), U2.8 (GND)
- net col0: now also U2.4 (GP2)
- net col1: now also U2.7 (GP5)
- net col2: now also U2.6 (GP4)
- net col3: now also U2.10 (GP7)
- net col4: now also U2.11 (GP8)
- net col5: now also U2.12 (GP9)
- net rowA: now also U2.5 (GP3)
- net rowB: now also U2.9 (GP6)
- net rowC: now also U2.16 (GP12)
- net rowD: now also U2.17 (GP13)
- net rowE: now also U2.19 (GP14)
- net LED_L: no longer names the net of U1.20 (GP15)
- net LED_L: no longer D10.2 (A)
- new net: D60.1 (K), R4.1
- new net: D59.1 (K), R3.1
- new net CAPS_LOCK: D59.2 (A), U2.25 (GP19)
- new net NUM_LOCK: D10.2 (A), U2.26 (GP20)
- new net RST_R: SW30.1, U2.30 (RUN)
- new net RX_R: J3.B, U2.2RXL (GP1/RX)
- new net SCROLL_LOCK: D60.2 (A), U2.24 (GP18)
- new net TX_R: J3.C, U2.1TXL (GP0/TX)
- new net Vin_R: J3.DR, U2.39 (Vin)
- new net Vout_R: J3.DL, U2.40 (Vout)
- no-connect marks 11 -> 21
Other:
- moved on the sheet: D10, J1, J2, R1, SW1, U1

Commit message: wip
Parts:
- removed D58: D_Small, symbol Device:D_Small
- removed J1, J3: TRRS, _tergo_lib:MJ-4PP-9, symbol _tergo_lib:MJ-4PP-9
- added D43: D_Small, symbol Device:D_Small
- added J1, J3: TRRS_SOCKET, _tergo_lib:MJ-4PP-9, symbol _tergo_lib:TRRS_SOCKET
- added J12, J13, J14, J15, J18, J19, J20, J21, J22, J23, J24, J25, J26, J27, J28, J29, J30, J31, J32, J33, J34, J35: Conn_01x01_Socket, _tergo_lib:THT_PAD, symbol Connector:Conn_01x01_Socket
- added J4, J5: Conn_01x06, symbol Connector_Generic:Conn_01x06
- added J6, J7: Conn_01x05, symbol Connector_Generic:Conn_01x05
- D10: value LED_Small -> NL
- D59: value LED_Small -> CL
- D60: value LED_Small -> SL
- J2: footprint Connector_PinHeader_2.54mm:PinHeader_1x04_P2.54mm_Vertical -> Connector_PinSocket_2.54mm:PinSocket_1x04_P2.54mm_Vertical
- U1, U2: symbol _tergo_lib:Raspberry_Pi_Pico -> _tergo_lib:Raspberry_Pi_Pico_choc
Connections:
- net DISPLAY_SCL: no longer U2.22 (GP17/SCL)
- net DISPLAY_SDA: no longer U2.21 (GP16/SDA)
- net GND: now also J1.A, J3.A; no longer U1.29 (GP22)
- net RX_R: now also U2.2 (GP1/RX), J3.C; no longer U2.2RXL (GP1/RX)
- net TX_R: now also U2.1 (GP0/TX), J3.D; no longer U2.1TXL (GP0/TX)
- net at D50.2 (A): now also SW51.1; no longer SW50.1
- net at D48.2 (A): now also SW49.1; no longer SW48.1
- net at D45.2 (A): now also SW46.1; no longer SW45.1
- net at SW58.1: now also D57.2 (A)
- net at SW55.1: now also D54.2 (A); no longer D55.2 (A)
- net at D47.2 (A): now also SW48.1; no longer SW47.1
- net at D51.2 (A): now also SW52.1; no longer SW51.1
- net at SW56.1: now also D55.2 (A); no longer D56.2 (A)
- net at SW54.1: now also D53.2 (A); no longer D54.2 (A)
- net at D52.2 (A): now also SW53.1; no longer SW52.1
- net at D44.2 (A): now also SW45.1; no longer SW44.1
- net at SW57.1: now also D56.2 (A); no longer D57.2 (A)
- net at D46.2 (A): now also SW47.1; no longer SW46.1
- net at D49.2 (A): now also SW50.1; no longer SW49.1
- net 3V3 renamed 3V3_L
- net 3V3_L: now also U1.29 (GP22); no longer U2.36 (3V3)
- removed net RX: U1.2RXL (GP1/RX)
- removed net TX: U1.1TXL (GP0/TX)
- net Vin: no longer names the net of U1.39 (Vin)
- net Vin_R renamed VIN_R
- net VIN_R: now also J3.B
- net Vout renamed VOUT_L
- net VOUT_L: now also J1.B
- net Vout_R: no longer names the net of U2.40 (Vout)
- net col0 renamed COL0_L
- net COL0_L: now also J12.1 (Pin_1), J4.1 (Pin_1); no longer SW31.2, SW32.2, SW33.2, SW34.2, SW35.2, U2.4 (GP2)
- net col1 renamed COL1_L
- net COL1_L: now also J15.1 (Pin_1), J4.2 (Pin_2); no longer SW36.2, SW37.2, SW38.2, SW39.2, U2.7 (GP5)
- net col2 renamed COL2_L
- net COL2_L: now also J14.1 (Pin_1), J4.3 (Pin_3); no longer SW40.2, SW41.2, SW42.2, SW43.2, U2.6 (GP4)
- net col3 renamed COL3_L
- net COL3_L: now also J19.1 (Pin_1), J4.4 (Pin_4); no longer SW44.2, SW45.2, SW46.2, SW47.2, SW48.2, U2.10 (GP7)
- net col4 renamed COL4_L
- net COL4_L: now also J20.1 (Pin_1), J4.5 (Pin_5); no longer SW49.2, SW50.2, SW51.2, SW52.2, SW53.2, U2.11 (GP8)
- net col5 renamed COL5_L
- net COL5_L: now also J21.1 (Pin_1), J4.6 (Pin_6); no longer SW54.2, SW55.2, SW56.2, SW57.2, SW58.2, U2.12 (GP9)
- net rowA renamed ROWA_L
- net ROWA_L: now also J13.1 (Pin_1), J6.5 (Pin_5); no longer D30.1 (K), D35.1 (K), D39.1 (K), D44.1 (K), D49.1 (K), D54.1 (K), U2.5 (GP3)
- net rowB renamed ROWB_L
- net ROWB_L: now also J18.1 (Pin_1), J6.4 (Pin_4); no longer D31.1 (K), D36.1 (K), D40.1 (K), D45.1 (K), D50.1 (K), D55.1 (K), U2.9 (GP6)
- net rowC renamed ROWC_L
- net ROWC_L: now also J22.1 (Pin_1), J6.3 (Pin_3); no longer D32.1 (K), D37.1 (K), D41.1 (K), D46.1 (K), D51.1 (K), D56.1 (K), U2.16 (GP12)
- net rowD renamed ROWD_L
- net ROWD_L: now also J23.1 (Pin_1), J6.2 (Pin_2); no longer D33.1 (K), D38.1 (K), D42.1 (K), D47.1 (K), D52.1 (K), D57.1 (K), U2.17 (GP13)
- net rowE renamed ROWE_L
- net ROWE_L: now also J24.1 (Pin_1), J6.1 (Pin_1); no longer D34.1 (K), D48.1 (K), D53.1 (K), U2.19 (GP14)
- new net: D43.2 (A), SW44.1
- new net COL0_R: J25.1 (Pin_1), J5.1 (Pin_1), SW31.2, SW32.2, SW33.2, SW34.2, SW35.2, U2.4 (GP2)
- new net COL1_R: J28.1 (Pin_1), J5.2 (Pin_2), SW36.2, SW37.2, SW38.2, SW39.2, U2.7 (GP5)
- new net COL2_R: J27.1 (Pin_1), J5.3 (Pin_3), SW40.2, SW41.2, SW42.2, SW43.2, U2.6 (GP4)
- new net COL3_R: J30.1 (Pin_1), J5.4 (Pin_4), SW44.2, SW45.2, SW46.2, SW47.2, SW48.2, U2.10 (GP7)
- new net COL4_R: J31.1 (Pin_1), J5.5 (Pin_5), SW49.2, SW50.2, SW51.2, SW52.2, SW53.2, U2.11 (GP8)
- new net COL5_R: J32.1 (Pin_1), J5.6 (Pin_6), SW54.2, SW55.2, SW56.2, SW57.2, SW58.2, U2.12 (GP9)
- new net ROWA_R: D30.1 (K), D35.1 (K), D39.1 (K), D43.1 (K), D48.1 (K), D53.1 (K), J26.1 (Pin_1), J7.5 (Pin_5), U2.5 (GP3)
- new net ROWB_R: D31.1 (K), D36.1 (K), D40.1 (K), D44.1 (K), D49.1 (K), D54.1 (K), J29.1 (Pin_1), J7.4 (Pin_4), U2.9 (GP6)
- new net ROWC_R: D32.1 (K), D37.1 (K), D41.1 (K), D45.1 (K), D50.1 (K), D55.1 (K), J33.1 (Pin_1), J7.3 (Pin_3), U2.16 (GP12)
- new net ROWD_R: D33.1 (K), D38.1 (K), D42.1 (K), D46.1 (K), D51.1 (K), D56.1 (K), J34.1 (Pin_1), J7.2 (Pin_2), U2.17 (GP13)
- new net ROWE_R: D34.1 (K), D47.1 (K), D52.1 (K), D57.1 (K), J35.1 (Pin_1), J7.1 (Pin_1), U2.19 (GP14)
- new net RX_L: J1.D, U1.2 (GP1/RX)
- new net TX_L: J1.C, U1.1 (GP0/TX)
- no-connect marks 21 -> 27
Other:
- moved on the sheet: D10, D59, D60, J2, R1, R3, R4, U1, U2

Commit message: wip
Parts:
- removed SW1: SW_Push, symbol Switch:SW_Push
- added H1, H2, H3, H4, H5, H6, H7, H8: MountingHole, _tergo_lib:MountHole_5mm, symbol Mechanical:MountingHole
- added SW1: RST_LEFT, _tergo_lib:pushbutton-THT-2pin, symbol Switch:SW_Push_Dual_x2
- SW30: value SW_Push -> RST_RIGHT; footprint (none) -> _tergo_lib:pushbutton-THT-2pin; symbol Switch:SW_Push -> Switch:SW_Push_Dual_x2
Connections:
- net GND: now also SW1.2 (D); no longer U2.13 (GND), U2.18 (GND), U2.3 (GND), U2.8 (GND)
- net RST_L: now also SW1.1 (C)
- no-connect marks 27 -> 31
